File: KiCAD_Files/PCB.kicad_pcb (KiCad board)
At the start: 2 copper layers, 73.7 x 48.3 mm, 41 parts, among them SW1 SW_Push, SW2 SW_Push, SW3 SW_Push, U1 NodeMCU_1.0_(ESP-12E), U2 LM35-LP

Commit message: Some residual changes from last commit
Parts:
- added R14: 1k, Resistor_THT:R_Axial_DIN0207_L6.3mm_D2.5mm_P7.62mm_Horizontal, F.Cu at (146.6, 53.7)
- added SMD-D1: KCSC02-105, Display_7Segment:KCSC02-105, F.Cu at (176.5, 65.4)
- added SMD-D2: LED_RKGB, LED_THT:LED_D5.0mm-4_RGB_Staggered_Pins, F.Cu at (144.8, 28.6)
- added SMD-R14: 1k, Resistor_SMD:R_1206_3216Metric_Pad1.30x1.75mm_HandSolder, F.Cu at (149.6, 48.8)
- added SMD-SW1: SW_Push, Button_Switch_SMD:SW_Push_1P1T_NO_6x6mm_H9.5mm, F.Cu at (230.5, 64.1)
- added SMD-SW2: SW_Push, Button_Switch_SMD:SW_Push_1P1T_NO_6x6mm_H9.5mm, F.Cu at (230.5, 51.4)
- added SMD-SW3: SW_Push, Button_Switch_SMD:SW_Push_1P1T_NO_6x6mm_H9.5mm, F.Cu at (230.5, 39.4)
- added SMD-U1: MCP9700T-ETT, Package_TO_SOT_SMD:SOT-23, F.Cu at (220.6, 51.3)
- R10, R9: footprint Resistor_THT:R_Axial_DIN0207_L6.3mm_D2.5mm_P7.62mm_Horizontal -> Resistor_THT:R_Axial_DIN0207_L6.3mm_D2.5mm_P10.16mm_Horizontal
- R12, R13: footprint Resistor_THT:R_Axial_DIN0207_L6.3mm_D2.5mm_P10.16mm_Horizontal -> Resistor_THT:R_Axial_DIN0207_L6.3mm_D2.5mm_P7.62mm_Horizontal
- turned SMD-R11 to 90 degrees
Connections:
- D1 pad 5: unconnected-(D1-Pad5) -> Net-(D1-Pad5)
- R10 pad 1: /SEGG -> +3V3
- R10 pad 2: Net-(D2-Pad4) -> /BT2
- R12 pad 1: +3V3 -> /SEGA
- R12 pad 2: /BT1 -> Net-(D2-Pad1)
- R13 pad 1: +3V3 -> /SEGD
- R13 pad 2: /BT2 -> Net-(D2-Pad3)
- R8 pad 1: /SEGA -> /SEGDP
- R8 pad 2: Net-(D2-Pad1) -> Net-(D1-Pad5)
- R9 pad 1: /SEGD -> +3V3
- R9 pad 2: Net-(D2-Pad3) -> /BT1
- SMD-R1 pad 2: Net-(D1-Pad7) -> Net-(SMD-D1-Pad7)
- SMD-R10 pad 1: /SEGG -> +3V3
- SMD-R10 pad 2: Net-(D2-Pad4) -> /BT2
- SMD-R11 pad 1: /BT3 -> +3V3
- SMD-R11 pad 2: +3V3 -> /BT3
- SMD-R12 pad 1: /BT1 -> /SEGA
- SMD-R12 pad 2: +3V3 -> Net-(SMD-D2-Pad1)
- SMD-R13 pad 1: /BT2 -> /SEGD
- SMD-R13 pad 2: +3V3 -> Net-(SMD-D2-Pad3)
- SMD-R2 pad 2: Net-(D1-Pad6) -> Net-(SMD-D1-Pad6)
- SMD-R3 pad 2: Net-(D1-Pad4) -> Net-(SMD-D1-Pad4)
- SMD-R4 pad 2: Net-(D1-Pad2) -> Net-(SMD-D1-Pad2)
- SMD-R5 pad 2: Net-(D1-Pad1) -> Net-(SMD-D1-Pad1)
- SMD-R6 pad 2: Net-(D1-Pad9) -> Net-(SMD-D1-Pad9)
- SMD-R7 pad 2: Net-(D1-Pad10) -> Net-(SMD-D1-Pad10)
- SMD-R8 pad 1: /SEGA -> /SEGDP
- SMD-R8 pad 2: Net-(D2-Pad1) -> Net-(SMD-D1-Pad5)
- SMD-R9 pad 1: /SEGD -> +3V3
- SMD-R9 pad 2: Net-(D2-Pad3) -> /BT1
