File: KiCAD_Files/Standard-S/PCB-S.kicad_sch (KiCad schematic)
At the start: 23 parts, among them J1 Conn_01x15_Female, J2 Conn_01x15_Female, SW1 SW_Push, SW2 SW_Push, SW3 SW_Push, U1 MCP9700AT-ETT

Commit message: Added Panelization files and stuff
Parts:
- removed D2: LED_RKGB, LED_THT:LED_D5.0mm-4_RGB_Staggered_Pins, symbol Device:LED_RKGB
- added D2: LED_RGB, LED_SMD:LED_RGB_5050-6, symbol Device:LED_RGB
Connections:
- net GND: now also D2.4 (BK), D2.5 (RK), D2.6 (GK)
- net at R11.2: now also D2.3 (BA)
- net at R9.2: now also D2.2 (RA)
- net at R10.2: now also D2.1 (GA)
Changed lines of the file:
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@@
   (junction (at 92.71 76.2) (diameter 1.016) (color 0 0 0 0))
   (junction (at 92.71 80.01) (diameter 1.016) (color 0 0 0 0))
+  (junction (at 128.27 57.15) (diameter 1.016) (color 0 0 0 0))
+  (junction (at 128.27 62.23) (diameter 1.016) (color 0 0 0 0))
   (junction (at 130.81 80.01) (diameter 1.016) (color 0 0 0 0))
   (junction (at 130.81 83.82) (diameter 1.016) (color 0 0 0 0))
@@
     (stroke (width 0) (type solid) (color 0 0 0 0))
   )
+  (wire (pts (xy 125.73 52.07) (xy 128.27 52.07))
+    (stroke (width 0) (type solid) (color 0 0 0 0))
+  )
+  (wire (pts (xy 125.73 62.23) (xy 128.27 62.23))
+    (stroke (width 0) (type solid) (color 0 0 0 0))
+  )
+  (wire (pts (xy 128.27 52.07) (xy 128.27 57.15))
+    (stroke (width 0) (type solid) (color 0 0 0 0))
+  )
   (wire (pts (xy 128.27 57.15) (xy 125.73 57.15))
     (stroke (width 0) (type solid) (color 0 0 0 0))
   )
-  (wire (pts (xy 128.27 59.69) (xy 128.27 57.15))
+  (wire (pts (xy 128.27 62.23) (xy 128.27 57.15))
+    (stroke (width 0) (type solid) (color 0 0 0 0))
+  )
+  (wire (pts (xy 128.27 66.04) (xy 128.27 62.23))
     (stroke (width 0) (type solid) (color 0 0 0 0))
   )
@@
     (pin "1")
   )
-  (symbol (lib_id "power:GND") (at 128.27 59.69 0) (unit 1)
-    (in_bom yes) (on_board yes)
-    (property "Reference" "#PWR02" (id 0) (at 128.27 66.04 0)
-      (effects (font (size 1.27 1.27)) hide)
-    )
-    (property "Value" "GND" (id 1) (at 128.3843 64.0144 0))
-    (property "Footprint" "" (id 2) (at 128.27 59.69 0)
-      (effects (font (size 1.27 1.27)) hide)
-    )
-    (property "Datasheet" "" (id 3) (at 128.27 59.69 0)
+  (symbol (lib_id "power:GND") (at 128.27 66.04 0) (unit 1)
+    (in_bom yes) (on_board yes)
+    (property "Reference" "#PWR02" (id 0) (at 128.27 72.39 0)
+      (effects (font (size 1.27 1.27)) hide)
+    )
+    (property "Value" "GND" (id 1) (at 128.3843 70.3644 0))
+    (property "Footprint" "" (id 2) (at 128.27 66.04 0)
+      (effects (font (size 1.27 1.27)) hide)
+    )
+    (property "Datasheet" "" (id 3) (at 128.27 66.04 0)
       (effects (font (size 1.27 1.27)) hide)
     )
@@
     (pin "3")
   )
-  (symbol (lib_id "Device:LED_RKGB") (at 120.65 57.15 0) (mirror y) (unit 1)
-    (in_bom yes) (on_board yes)
-    (property "Reference" "D2" (id 0) (at 120.65 46.99 0))
-    (property "Value" "LED_RKGB" (id 1) (at 129.54 54.61 0)
-      (effects (font (size 1.27 1.27)) hide)
-    )
-    (property "Footprint" "LED_THT:LED_D5.0mm-4_RGB_Staggered_Pins" (id 2) (at 120.65 58.42 0)
+  (symbol (lib_id "Device:LED_RGB") (at 120.65 57.15 0) (mirror y) (unit 1)
+    (in_bom yes) (on_board yes)
+    (property "Reference" "D2" (id 0) (at 115.57 50.8 0))
+    (property "Value" "LED_RGB" (id 1) (at 120.65 46.99 0)
+      (effects (font (size 1.27 1.27)) hide)
+    )
+    (property "Footprint" "LED_SMD:LED_RGB_5050-6" (id 2) (at 120.65 58.42 0)
       (effects (font (size 1.27 1.27)) hide)
     )
@@
       (effects (font (size 1.27 1.27)) hide)
     )
-    (pin "1")
-    (pin "2")
+    (pin "5")
+    (pin "6")
+    (pin "4")
     (pin "3")
-    (pin "4")
+    (pin "1")
+    (pin "2")
   )
   (symbol (lib_id "Connector:Conn_01x15_Female") (at 31.75 39.37 0) (unit 1)
@@
       (reference "D1") (unit 1) (value "SM420561N") (footprint "Display_7Segment:7SegmentLED_LTS6760_LTS6780")
     )
-    (path "/832d2faa-8705-4593-a62c-f437f8bbfe9a"
-      (reference "D2") (unit 1) (value "LED_RKGB") (footprint "LED_THT:LED_D5.0mm-4_RGB_Staggered_Pins")
+    (path "/bf320462-ceb3-484a-be42-234b95038eaf"
+      (reference "D2") (unit 1) (value "LED_RGB") (footprint "LED_SMD:LED_RGB_5050-6")
     )
     (path "/dd95e13a-2c59-4c92-b566-bcd681b2e7e9"
